Commit message: simplify collision body for sparkplug

File: description/models/sparkplug/sparkplug.urdf (robot description, URDF)
Before this commit: robot sparkplug, 1 links, 0 joints
Links:
- link sparkplug: geometry collision cylinder length=0.072 radius=0.009; visual mesh filename=model://sparkplug/meshes/visual/sparkplug.stl
