Commit message: added pick and insert demo

File: description/models/panda/panda.urdf (robot description, URDF)
Before this commit: robot panda, 14 links, 13 joints
Joints:
- joint panda_joint7: limit lower=-2.8973 upper=2.8973 effort=12 velocity=2.6100 -> lower=-3.15 upper=3.15 effort=12 velocity=2.6100

File: description/models/sparkplug/sparkplug.urdf (robot description, URDF)
Before this commit: robot sparkplug, 1 links, 0 joints
Links:
- link sparkplug: geometry collision box size=0.0127 0.0127 0.072; visual mesh filename=model://sparkplug/meshes/visual/sparkplug.stl

Commit message: pick and insert example sort of working

File: description/models/panda/panda.urdf (robot description, URDF)
Before this commit: robot panda, 14 links, 13 joints
Joints:
- joint panda_finger_joint1: limit lower=-0.001 upper=0.04 effort=20 velocity=0.3 -> lower=-0.001 upper=0.04 effort=100 velocity=0.3
- joint panda_finger_joint2: limit lower=-0.001 upper=0.04 effort=20 velocity=0.3 -> lower=-0.001 upper=0.04 effort=100 velocity=0.3

File: description/models/sparkplug/sparkplug.urdf (robot description, URDF)
Before this commit: robot sparkplug, 1 links, 0 joints
Links:
- link sparkplug: geometry collision cylinder length=0.072 radius=0.009; visual mesh filename=model://sparkplug/meshes/visual/sparkplug.stl

File: description/models/sparkplug_socket/sparkplug_socket.urdf (robot description, URDF)
Before this commit: robot sparkplug_socket, 1 links, 0 joints
Links:
- link sparkplug_socket: mass 2.673 -> 3.962

Commit message: reset finger joint effort limits

File: description/models/panda/panda.urdf (robot description, URDF)
Before this commit: robot panda, 14 links, 13 joints
Joints:
- joint panda_finger_joint1: limit lower=-0.001 upper=0.04 effort=100 velocity=0.3 -> lower=-0.001 upper=0.04 effort=20. velocity=0.3
- joint panda_finger_joint2: limit lower=-0.001 upper=0.04 effort=100 velocity=0.3 -> lower=-0.001 upper=0.04 effort=20. velocity=0.3
