Commit message: fixed rviz

File: description/models/kinect/kinect.urdf (robot description, URDF)
Before this commit: robot TestKinect, 6 links, 5 joints
Links:
- link camera_link: geometry collision box size=0.07271 0.27794 0.073; visual mesh filename=file://$(find panda_ros2_gazebo)/description/models/kinect/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
