Commit message: minor fixes

File: description/models/kinect/kinect.xacro (robot description, xacro)
@@ -1,8 +1,10 @@
 <?xml version="1.0" ?>
-<!-- =================================================================================== -->
-<!-- |    This document was autogenerated by xacro from kinect.urdf.xacro              | -->
-<!-- |    EDITING THIS FILE BY HAND IS NOT RECOMMENDED                                 | -->
-<!-- =================================================================================== -->
-<robot name="kinect" xmlns:xacro="http://www.ros.org/wiki/xacro">
+<robot xmlns:xacro="http://www.ros.org/wiki/xacro" name="kinect">
+  <xacro:property name="x" value="0.0" />
+  <xacro:property name="y" value="0.0" />
+  <xacro:property name="z" value="0.0" />
+  <xacro:property name="R" value="0.0" />
+  <xacro:property name="P" value="0.0" />
+  <xacro:property name="Y" value="0.0" />
   <link name="world"/>
   <!-- Microsoft Kinect / ASUS Xtion PRO Live for simulation -->
@@ -27,5 +29,5 @@
         <alwaysOn>true</alwaysOn>
         <updateRate>10.0</updateRate>
-        <robotNamespace>kinect</robotNamespace>
+        <!-- <robotNamespace>kinect</robotNamespace> -->
         <cameraName>camera1</cameraName>
         <imageTopicName>/camera/color/image_raw</imageTopicName>
@@ -48,5 +50,5 @@
   <!-- Parameterised in part by the values in kinect_properties.urdf.xacro -->
   <joint name="camera_rgb_joint" type="fixed">
-    <origin xyz="0 0 0" rpy="0 0 0"/>
+    <origin xyz="${x} ${y} ${z}" rpy="${R} ${P} ${Y}"/>
     <parent link="world"/>
     <child link="camera_rgb_frame"/>
