Commit message: rearranged repo and added package for custom messages, for some reason, node not spinning joint states callback

File: panda_control/description/models/kinect/kinect.xacro (robot description, xacro)
@@ -82,5 +82,5 @@
       <origin rpy="0 0 1.57079632679" xyz="0 0 0"/>
       <geometry>
-        <mesh filename="file://$(find panda_ros2_gazebo)/description/models/kinect/meshes/visual/kinect.dae"/>
+        <mesh filename="file://$(find panda_control)/description/models/kinect/meshes/visual/kinect.dae"/>
       </geometry>
     </visual>

File: panda_control/description/models/panda/panda.urdf (robot description, URDF)
Before this commit: robot panda, 14 links, 13 joints
Links:
- link panda_hand: geometry collision mesh filename=file://$(find panda_control)/description/models/panda/meshe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; visual mesh filename=file://$(find panda_control)/description/models/panda/meshe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
- link panda_leftfinger: geometry collision mesh filename=file://$(find panda_control)/description/models/panda/meshe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; visual mesh filename=file://$(find panda_control)/description/models/panda/meshe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
- link panda_link0: geometry collision mesh filename=file://$(find panda_control)/description/models/panda/meshe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; visual mesh filename=file://$(find panda_control)/description/models/panda/meshe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
- link panda_link1: geometry collision mesh filename=file://$(find panda_control)/description/models/panda/meshe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; visual mesh filename=file://$(find panda_control)/description/models/panda/meshe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
- link panda_link2: geometry collision mesh filename=file://$(find panda_control)/description/models/panda/meshe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; visual mesh filename=file://$(find panda_control)/description/models/panda/meshe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
- link panda_link3: geometry collision mesh filename=file://$(find panda_control)/description/models/panda/meshe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; visual mesh filename=file://$(find panda_control)/description/models/panda/meshe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
- link panda_link4: geometry collision mesh filename=file://$(find panda_control)/description/models/panda/meshe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; visual mesh filename=file://$(find panda_control)/description/models/panda/meshe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
- link panda_link5: geometry collision mesh filename=file://$(find panda_control)/description/models/panda/meshe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; visual mesh filename=file://$(find panda_control)/description/models/panda/meshe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
- link panda_link6: geometry collision mesh filename=file://$(find panda_control)/description/models/panda/meshe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; visual mesh filename=file://$(find panda_control)/description/models/panda/meshe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
- link panda_link7: geometry collision mesh filename=file://$(find panda_control)/description/models/panda/meshe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; visual mesh filename=file://$(find panda_control)/description/models/panda/meshe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
- link panda_rightfinger: geometry collision mesh filename=file://$(find panda_control)/description/models/panda/meshe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; visual mesh filename=file://$(find panda_control)/description/models/panda/meshe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
